File: 3k_badge_eda/3000_Society_Badge/3000_Society_Badge.kicad_pcb (KiCad board)
At the start: 2 copper layers, 1 part, among them IC1 Trinket3v3

Commit message: kicad-library-updates
Parts:
- added D1: WS2812B, 3000_Society_Badge:LED_WS2812B_PLCC4_5.0x5.0mm_P3.2mm, F.Cu at (106.6, 116.2)
- IC1: value Trinket3v3 -> Trinket_M0_3v3
- moved IC1 12.4 mm to (142.1, 94.3)
Changed lines of the file:
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@@
     (tracks 0)
     (zones 0)
-    (modules 1)
-    (nets 11)
+    (modules 2)
+    (nets 15)
   )
   (page A4)
@@
     (pad_to_mask_clearance 0.2)
     (aux_axis_origin 0 0)
-    (visible_elements FFFFFF7F)
+    (visible_elements 7FFFFFFF)
     (pcbplotparams
       (layerselection 0x00030_80000001)
@@
   (net 9 "Net-(IC1-Pad9)")
   (net 10 "Net-(IC1-Pad10)")
+  (net 11 "Net-(D1-Pad3)")
+  (net 12 "Net-(D1-Pad4)")
+  (net 13 "Net-(D1-Pad2)")
+  (net 14 "Net-(D1-Pad1)")
   (net_class Default "This is the default net class."
     (clearance 0.2)
@@
     (uvia_dia 0.3)
     (uvia_drill 0.1)
+    (add_net "Net-(D1-Pad1)")
+    (add_net "Net-(D1-Pad2)")
+    (add_net "Net-(D1-Pad3)")
+    (add_net "Net-(D1-Pad4)")
     (add_net "Net-(IC1-Pad1)")
     (add_net "Net-(IC1-Pad10)")
@@
     (add_net "Net-(IC1-Pad9)")
   )
+  (module 3000_Society_Badge:LED_WS2812B_PLCC4_5.0x5.0mm_P3.2mm (layer F.Cu)
+    (at 106.6038 116.1796)
+    (descr https://cdn-shop.adafruit.com/datasheets/WS2812B.pdf)
+    (tags "LED RGB NeoPixel")
+    (attr smd)
+    (fp_text reference D1 (at 0 -3.5) (layer F.SilkS)
+      (effects (font (size 1 1) (thickness 0.15)))
+    )
+    (fp_text value WS2812B (at 0 4) (layer F.Fab)
+      (effects (font (size 1 1) (thickness 0.15)))
+    )
+    (fp_text user 1 (at -4.15 -1.6) (layer F.SilkS)
+      (effects (font (size 1 1) (thickness 0.15)))
+    )
+    (fp_text user %R (at 0 0) (layer F.Fab)
+      (effects (font (size 0.8 0.8) (thickness 0.15)))
+    )
+    (fp_line (start 3.45 -2.75) (end -3.45 -2.75) (layer F.CrtYd) (width 0.05))
+    (fp_line (start 3.45 2.75) (end 3.45 -2.75) (layer F.CrtYd) (width 0.05))
+    (fp_line (start -3.45 2.75) (end 3.45 2.75) (layer F.CrtYd) (width 0.05))
+    (fp_line (start -3.45 -2.75) (end -3.45 2.75) (layer F.CrtYd) (width 0.05))
+    (fp_line (start 2.5 1.5) (end 1.5 2.5) (layer F.Fab) (width 0.1))
+    (fp_line (start -2.5 -2.5) (end -2.5 2.5) (layer F.Fab) (width 0.1))
+    (fp_line (start -2.5 2.5) (end 2.5 2.5) (layer F.Fab) (width 0.1))
+    (fp_line (start 2.5 2.5) (end 2.5 -2.5) (layer F.Fab) (width 0.1))
+    (fp_line (start 2.5 -2.5) (end -2.5 -2.5) (layer F.Fab) (width 0.1))
+    (fp_line (start -3.65 -2.75) (end 3.65 -2.75) (layer F.SilkS) (width 0.12))
+    (fp_line (start -3.65 2.75) (end 3.65 2.75) (layer F.SilkS) (width 0.12))
+    (fp_line (start 3.65 2.75) (end 3.65 1.6) (layer F.SilkS) (width 0.12))
+    (fp_circle (center 0 0) (end 0 -2) (layer F.Fab) (width 0.1))
+    (pad 3 smd rect (at 2.45 1.6) (size 1.5 1) (layers F.Cu F.Paste F.Mask)
+      (net 11 "Net-(D1-Pad3)"))
+    (pad 4 smd rect (at 2.45 -1.6) (size 1.5 1) (layers F.Cu F.Paste F.Mask)
+      (net 12 "Net-(D1-Pad4)"))
+    (pad 2 smd rect (at -2.45 1.6) (size 1.5 1) (layers F.Cu F.Paste F.Mask)
+      (net 13 "Net-(D1-Pad2)"))
+    (pad 1 smd rect (at -2.45 -1.6) (size 1.5 1) (layers F.Cu F.Paste F.Mask)
+      (net 14 "Net-(D1-Pad1)"))
+    (model ${KISYS3DMOD}/LED_SMD.3dshapes/LED_WS2812B_PLCC4_5.0x5.0mm_P3.2mm.wrl
+      (at (xyz 0 0 0))
+      (scale (xyz 1 1 1))
+      (rotate (xyz 0 0 0))
+    )
+  )
   (module 3000_Society_Badge:Trinket_3v3 (layer F.Cu)
-    (at 148.5011 105.0036)
+    (at 142.1384 94.3102)
     (descr "IC, Adafruit, Trinket M0, 3v3, Trinket3v3")
     (tags "IC Adafruit Trinket M0 3v3 Trinket3v3")
@@
       (effects (font (size 1 1) (thickness 0.15)))
     )
-    (fp_text value Trinket3v3 (at 0 6.985) (layer F.Fab)
+    (fp_text value Trinket_M0_3v3 (at 0 6.985) (layer F.Fab)
       (effects (font (size 1 1) (thickness 0.15)))
     )
