File: 3k_badge_eda/3000_Society_Badge_K5/3000_Society_Badge_K5.kicad_pcb (KiCad board)
At the start: 2 copper layers, 195.2 x 165.9 mm, 28 parts, among them IC1 Trinket_M0

Commit message: corrections from 1st prototype run
Parts:
- C1, C2, C3, C4, C5: value CP 100uF -> 100uF
- R1, R10, R2, R20, R4, R40, R5: value R 470ohm -> 470 ohm; footprint 3000_Society_Badge:R_Axial_DIN0204_L3.6mm_D1.6mm_P5.08mm_Horizontal -> 3000_Society_Badge:R_Axial_DIN0207_L6.3mm_D2.5mm_P7.62mm_Horizontal
- R3: value R 470ohm -> 100 ohm; footprint 3000_Society_Badge:R_Axial_DIN0204_L3.6mm_D1.6mm_P5.08mm_Horizontal -> 3000_Society_Badge:R_Axial_DIN0207_L6.3mm_D2.5mm_P7.62mm_Horizontal
- moved R40 6.83 mm to (180.0, 67.7), turned to 270 degrees
- moved R10 2.95 mm to (120.8, 93.7)
- moved R2 1.15 mm to (113.4, 99.7)
- moved R5 0.89 mm to (145.5, 82.9)
- moved R1 0.68 mm to (115.9, 98.7)
- moved R3 0.19 mm to (140.8, 84.8)
- turned R20 to 28 degrees
Routing:
- net Net-(IC1-Pad3): track 8.78 -> 12.8 mm
- net Net-(C5-Pad1): track 109.1 -> 112.3 mm
- net Net-(C1-Pad1): track 174.2 -> 171.6 mm
- net Net-(C2-Pad1): track 180.4 -> 183.0 mm
- net Net-(C4-Pad1): track 114.7 -> 117.2 mm
- net Net-(C3-Pad1): track 119.0 -> 116.5 mm
- net Net-(IC1-Pad10): track 138.4 -> 139.9 mm
- net Net-(D20-Pad4): track 9.25 -> 7.95 mm
- net Net-(IC1-Pad8): track 74.2 -> 73.5 mm
- net Net-(D40-Pad4): track 4.84 -> 4.29 mm
Other:
- outline, holes or cut-outs redrawn
- board text added: "https://3000society.com/"
